Commit message: Got OMPL planner directly.

File: urdf/bot.urdf (robot description, URDF)
Before this commit: robot bubblebot, 1 links, 0 joints
Links:
- link base_link: geometry collision cylinder length=0.2 radius=0.2; visual cylinder length=0.2 radius=0.2

Commit message: Got re-planning sorta working? Planning still pretty bad.

File: urdf/bot.urdf (robot description, URDF)
Before this commit: robot bubblebot, 1 links, 0 joints
Links:
- link base_link: geometry collision cylinder length=0.1 radius=0.25; visual cylinder length=0.2 radius=0.2

Commit message: Small improvements.

File: urdf/bot.urdf (robot description, URDF)
Before this commit: robot bubblebot, 1 links, 0 joints
Links:
- link base_link: geometry collision cylinder length=0.1 radius=0.25; visual box size=0.36 0.36 0.05

Commit message: Progress!

File: urdf/bot.urdf (robot description, URDF)
Before this commit: robot bubblebot, 1 links, 0 joints
Links:
- added link end_effector; visual sphere radius=0.05
- link base_link: geometry collision box size=0.01 0.5 0.01; collision cylinder length=0.1 radius=0.25
Joints:
- added joint stick: type fixed, parent base_link, child end_effector, origin xyz=0.0 0.6750 0.0
